File: pcb/mem_pmod/mem_pmod.kicad_sch (KiCad schematic)
At the start: 4 parts, among them J1 Conn_01x04_Pin

Commit message: continue working on schematic
Parts:
- added Clock_Divider: SY100EP32VKG, MSOP-8_K8-1_MCL, symbol SY100EP32VKG:SY100EP32VKG
- added Flash: W25Q128JVSIM, SOIC_128JVSIM_WIN, symbol W25Q128JVSIM:W25Q128JVSIM
- added RAM0, RAM1, RAM2, VRAM0, VRAM1: APS6404L-3SQR-SN, APS6404L-3SQR-SN_APY, symbol ul_APS6404L-3SQR-SN:APS6404L-3SQR-SN
- added U1: 74HC125D, SOIC14_TOS, symbol 74HC125D:74HC125D
- added VGA_DFLIP (x2): SN74HC374NSR, NS20, symbol SN74HC374NSR:SN74HC374NSR
Connections:
- net DEMUX_CS3: now also NOT.13 (6A)
- net DEMUX_VS0: now also NOT.11 (5A)
- net DEMUX_VS1: now also NOT.9 (4A)
- net GND: now also Clock_Divider.5 (VEE), Flash.4 (GND), RAM0.8 (VDD), RAM1.8 (VDD), RAM2.8 (VDD), U1.7 (GND), VGA_DFLIP.10 (GND), VGA_DFLIP.10 (GND), VRAM0.8 (VDD), VRAM1.8 (VDD)
- net PMOD_A0: now also Flash.5 (DI_(IO0)), RAM0.5 (SI/SIO[0]), RAM1.5 (SI/SIO[0]), RAM2.5 (SI/SIO[0])
- net PMOD_A1: now also Flash.2 (DO_(IO1)), RAM0.2 (SO/SIO[1]), RAM1.2 (SO/SIO[1]), RAM2.2 (SO/SIO[1])
- net PMOD_A2: now also Flash.3 (/WP_(IO2)), RAM0.3 (SIO[2]), RAM1.3 (SIO[2]), RAM2.3 (SIO[2])
- net PMOD_A3: now also Flash.7 (HOLD(IO3)), RAM0.7 (SIO[3]), RAM1.7 (SIO[3]), RAM2.7 (SIO[3])
- net PMOD_B0: now also VRAM0.5 (SI/SIO[0]), VRAM1.5 (SI/SIO[0])
- net PMOD_B1: now also VRAM0.2 (SO/SIO[1]), VRAM1.2 (SO/SIO[1])
- net PMOD_B2: now also VRAM0.3 (SIO[2]), VRAM1.3 (SIO[2])
- net PMOD_B3: now also VRAM0.7 (SIO[3]), VRAM1.7 (SIO[3])
- net PRJ_Clock: now also Clock_Divider.2 (CLK), Flash.6 (CLK), RAM0.6 (SCLK), RAM1.6 (SCLK), RAM2.6 (SCLK), VRAM0.6 (SCLK), VRAM1.6 (SCLK)
- net RAM_CS0: now also RAM0.1 (/CE)
- net RAM_CS1: now also RAM1.1 (/CE)
- net VCC: now also Clock_Divider.8 (VCC), Flash.8 (VCC), RAM0.4 (VSS), RAM1.4 (VSS), RAM2.4 (VSS), U1.14 (VCC), VGA_DFLIP.1 (*OE), VGA_DFLIP.1 (*OE), VGA_DFLIP.20 (VCC), VGA_DFLIP.20 (VCC), VRAM0.4 (VSS), VRAM1.4 (VSS)
- net RAM_VS0: now reaches NOT.10 (5Y)
- net RAM_VS0: now also VRAM0.1 (/CE)
- net RAM_CS3: now reaches NOT.12 (6Y)
- net RAM_CS3: now also Flash.1 (/CS)
- net RAM_CS2: now reaches NOT.6 (3Y)
- net RAM_CS2: now also RAM2.1 (/CE)
- net RAM_VS1: now reaches NOT.8 (4Y)
- net RAM_VS1: now also VRAM1.1 (/CE)
- new net DIV_CLK_0: Clock_Divider.7 (Q), VGA_DFLIP.11 (CLK)
- new net DIV_CLK_1: Clock_Divider.6 (*Q), VGA_DFLIP.11 (CLK)
